File: upuaut.sch (KiCad schematic (older format))
At the start: 1 part

Commit message: First Session
Parts:
- added Murata-Ceramic-Capacitor-50v1: C, symbol Device:C
- added U1: LDH-45B-1050, symbol OpenSourceCelluloid:LDH-45B-1050
- added U2: POTENTIOMETER, symbol OpenSourceCelluloid:POTENTIOMETER
- added U3: OKI-78SR-12v, symbol OpenSourceCelluloid:OKI-78SR-12v
- added U4: TMC2660-BOB-SOCKET, symbol OpenSourceCelluloid:TMC2660-BOB-SOCKET
- added U5: Connector-LED, symbol OpenSourceCelluloid:Connector-LED
- added U6: Motor-Connector, symbol OpenSourceCelluloid:Motor-Connector
- gave numbers to parts that had none: 1
Connections:
- net 3,3V: now reaches XA1.3V3 (3.3V)
- net 5V: now reaches XA1.5V
- net 5V: now also U2.1 (5V), U4.1 (VCC_IO)
- net CHIP-SELECT: now reaches XA1.D10 (D10_CS)
- net CHIP-SELECT: now also U4.6 (CSN)
- net MOSI-SDI: now reaches XA1.D11 (D11_MOSI)
- net MOSI-SDI: now also U4.4 (SDI)
- net MISO-SDO: now reaches XA1.D12 (D12_MISO)
- net MISO-SDO: now also U4.3 (SDO)
- net CLOCK: now reaches XA1.D13 (D13_SCK)
- net CLOCK: now also U4.5 (SCK), U4.9 (CLK16)
- net DIRECTION: now reaches XA1.D4
- net DIRECTION: now also U4.12 (DIR)
- net STEP: now reaches XA1.D5
- net STEP: now also U4.13 (STEP)
- net ENABLE: now reaches XA1.D6
- net ENABLE: now also U4.8 (DRV_ENV)
- net GND: now reaches XA1.GND1 (GND)
- net GND: now also XA1.GND2 (GND), Murata-Ceramic-Capacitor-50v1.2, U1.2 (VIN-), U1.3 (DIM-), U2.3 (GND), U3.2 (GND), U4.10 (SG_TST), U4.11 (GND), U4.14 (GND), U4.19 (GND), U4.2 (GND), U4.7 (GND)
- net 12V: now reaches XA1.VIN
- net 12V: now also U3.3 (VOUT)
- new net +24V: Murata-Ceramic-Capacitor-50v1.1, U1.1 (VIN), U3.1 (VIN), U4.20 (VS)
- new net BLACK: U4.15 (B2), U6.4 (BLACK)
- new net BLUE: U4.17 (A2), U6.2 (BLUE)
- new net GREEN: U4.16 (B1), U6.3 (GREEN)
- new net LED+: U1.7 (VOUT+), U5.1 (+)
- new net LED-: U1.6 (VOUT-), U5.2 (-)
- new net POTI: U1.4 (A-DIM), U2.2 (SIGNAL)
- new net RED: U4.18 (A1), U6.1 (RED)
- no-connect marks 0 -> 1
Other:
- moved on the sheet: XA1
